Commit message: updated robot urdf with camera

File: area54/urdf/area54.urdf (robot description, URDF)
Before this commit: robot area54, 5 links, 4 joints
Links:
- added link photo_link, mass 0.2; collision box size=0.05 0.05 0.05; visual box size=0.05 0.05 0.05
- link L_link: mass 1 -> 3
- link R_link: mass 1 -> 3
- link grip_link: mass 1 -> 0.8
Joints:
- added joint photo_joint: type fixed, parent base_link, child photo_link, origin xyz=-0.25 0 0.3 rpy=1.5708 0 0, axis 0 0 0
- joint grip_joint: axis 1 0 0 -> 0 0 -1; limit lower=0 upper=1.57 effort=2000 velocity=0.5 -> lower=0 upper=1.7 effort=3000 velocity=0.8; origin xyz=0.09 0.05 0.05 rpy=1.583 0 1.5708 -> xyz=0.181 0.22 0.02 rpy=1.5708 0.0033621 1.5708; type continuous -> revolute
